File: Diseño placa/Tearis.kicad_pcb (KiCad board)
At the start: 2 copper layers, 50 x 91.5 mm, 4 parts, among them M1 4056E_Loader_prot, M2 DC_DC_boost_module

Commit message: actualizacion diseño
Parts:
- removed M1: 4056E_Loader_prot, misc_footprints:4056E_LiIon_loader_SMT
- removed M2: DC_DC_boost_module, misc_footprints:XL6009_module_SMT
- removed REF**: Raspberry_Pi_Zero_Socketed_THT_FaceDown_MountingHoles, Module:Raspberry_Pi_Zero_Socketed_THT_FaceDown_MountingHoles
- removed REF**: PinHeader_1x02_P2.54mm_Vertical, Connector_PinHeader_2.54mm:PinHeader_1x02_P2.54mm_Vertical
- added TP1: ~, Custom_Footprints:TP4056-18650, F.Cu at (102.2, 116.4)
- added U1: RASPBERRY_PI_ZERO_2_W, Module:Raspberry_Pi_Zero_Socketed_THT_FaceDown_MountingHoles, F.Cu at (179.1, 87.5)
- added V1: 3.7, Connector_PinHeader_2.54mm:PinHeader_1x02_P2.54mm_Vertical, F.Cu at (110.7, 87.2)
- added xl1: ~, misc_footprints:XL6009_module, F.Cu at (175.0, 111.7)
Routing:
- net (no net): track 109.5 -> 0.00 mm
- net Net-(TP1-OUT_+): track 0.00 -> 42.7 mm
- net Net-(U1-5V_2): track 0.00 -> 37.0 mm
- net Net-(TP1-VOUT_-): track 0.00 -> 24.3 mm
- net GND: track 0.00 -> 6.93 mm
- net Net-(TP1-B_+): track 0.00 -> 5.89 mm
- net Net-(TP1-B_-): track 0.00 -> 5.23 mm
- removed copper zone on F.Cu, net (none)
Other:
- board size 50 x 91.5 mm -> 90 x 39 mm

Commit message: actualización placa
Parts:
- added SW1: SW_Push_Open, TestPoint:TestPoint_2Pads_Pitch5.08mm_Drill1.3mm, F.Cu at (108.5, 82.5)
- moved TP1 0.75 mm to (102.2, 117.1)
Connections:
- TP1 pad 3: Net-(TP1-OUT_+) -> Net-(SW1-A)
- TP1 pad 4: Net-(TP1-VOUT_-) -> Net-(TP1-B_+)
- TP1 pad 5: Net-(TP1-B_+) -> Net-(TP1-B_-)
- TP1 pad 6: Net-(TP1-B_-) -> Net-(TP1-VOUT_-)
- xl1 pad 1: Net-(TP1-OUT_+) -> Net-(SW1-B)
Routing:
- net Net-(TP1-OUT_+): track 42.7 -> 0.00 mm
- net Net-(SW1-B): track 0.00 -> 25.2 mm
- net Net-(SW1-A): track 0.00 -> 13.2 mm
- net Net-(TP1-B_-): track 5.23 -> 5.98 mm
- net Net-(TP1-B_+): track 5.89 -> 6.64 mm
- added copper zone on B.Cu, net GND
